File: _autosave-sdvx-pcb.kicad_sch (KiCad schematic)
At the start: 14 parts, among them U1 ATmega32U4-A

Commit message: some edits
some edits
Parts:
- added J?: AVR-ISP-6, symbol Connector:AVR-ISP-6
Changed lines of the file:
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@@
     (pin "1")
+  )
+  (symbol (lib_id "Connector:AVR-ISP-6") (at 170.18 118.11 0) (unit 1)
+    (in_bom yes) (on_board yes) (fields_autoplaced)
+    (property "Reference" "J?" (id 0) (at 161.29 115.5699 0)
+      (effects (font (size 1.27 1.27)) (justify right))
+    )
+    (property "Value" "AVR-ISP-6" (id 1) (at 161.29 118.1099 0)
+      (effects (font (size 1.27 1.27)) (justify right))
+    )
+    (property "Footprint" "" (id 2) (at 163.83 116.84 90)
+      (effects (font (size 1.27 1.27)) hide)
+    )
+    (property "Datasheet" " ~" (id 3) (at 137.795 132.08 0)
+      (effects (font (size 1.27 1.27)) hide)
+    )
+    (pin "1")
+    (pin "2")
+    (pin "3")
+    (pin "4")
+    (pin "5")
+    (pin "6")
   )
   (symbol (lib_id "Device:R_Small") (at 260.35 105.41 90) (unit 1)
@@
       (reference "C?") (unit 1) (value "0.1u") (footprint "")
     )
+    (path "/4d6c7527-0e60-407c-832c-7d63069963f4"
+      (reference "J?") (unit 1) (value "AVR-ISP-6") (footprint "")
+    )
     (path "/5ac495ab-2b20-4576-9f23-ecf5047bc209"
