File: sdvx-pcb.kicad_pcb (KiCad board)
At the start: 2 copper layers, 0 parts

Commit message: pcb start
start pcb
Parts:
- added BT-A1: MX-NoLED, MX_Only:MXOnly-1.5U-Hotswap, F.Cu at (95.4, 105.6)
- added BT-B1: MX-NoLED, MX_Only:MXOnly-1.5U-Hotswap, F.Cu at (130.2, 105.6)
- added BT-C1: MX-NoLED, MX_Only:MXOnly-1.5U-Hotswap, F.Cu at (164.9, 105.6)
- added BT-D1: MX-NoLED, MX_Only:MXOnly-1.5U-Hotswap, F.Cu at (200.0, 105.6)
- added C1: 22p, Capacitor_SMD:C_0805_2012Metric_Pad1.18x1.45mm_HandSolder, F.Cu at (238.4, 60.8)
- added C2: 0.1u, Capacitor_SMD:C_0805_2012Metric_Pad1.18x1.45mm_HandSolder, F.Cu at (210.6, 66.8)
- added C3: 0.1u, Capacitor_SMD:C_0805_2012Metric_Pad1.18x1.45mm_HandSolder, F.Cu at (204.7, 70.1)
- added C4: 22p, Capacitor_SMD:C_0805_2012Metric_Pad1.18x1.45mm_HandSolder, F.Cu at (215.4, 66.8)
- added C5: 0.1u, Capacitor_SMD:C_0805_2012Metric_Pad1.18x1.45mm_HandSolder, F.Cu at (214.3, 69.8)
- added C6: 0.1u, Capacitor_SMD:C_0805_2012Metric_Pad1.18x1.45mm_HandSolder, F.Cu at (209.5, 70.1)
- added C7: 1u, Capacitor_SMD:C_0805_2012Metric_Pad1.18x1.45mm_HandSolder, F.Cu at (220.2, 66.8)
- added FX-L1: MX-NoLED, MX_Only:MXOnly-2.25U-Hotswap, F.Cu at (112.7, 150.8)
- added FX-R1: MX-NoLED, MX_Only:MXOnly-2.25U-Hotswap, F.Cu at (182.6, 150.8)
- added Fe1: 500m, Fuse:Fuse_1206_3216Metric_Pad1.42x1.75mm_HandSolder, F.Cu at (205.2, 66.9)
- added J1: AVR-ISP-6, random-keyboard-parts:Reset_Pretty-Mask, F.Cu at (255.7, 47.7)
- added R1: 10k, Resistor_SMD:R_0805_2012Metric_Pad1.20x1.40mm_HandSolder, F.Cu at (229.8, 66.7)
- added R2: 5.1k, Resistor_SMD:R_0805_2012Metric_Pad1.20x1.40mm_HandSolder, F.Cu at (225.0, 66.7)
- added R3: 5.1k, Resistor_SMD:R_0805_2012Metric_Pad1.20x1.40mm_HandSolder, F.Cu at (238.3, 63.8)
- added R4: 22, Resistor_SMD:R_0805_2012Metric_Pad1.20x1.40mm_HandSolder, F.Cu at (223.8, 69.8)
- added R5: 22, Resistor_SMD:R_0805_2012Metric_Pad1.20x1.40mm_HandSolder, F.Cu at (278.8, 25.1)
- added R6: 10k, Resistor_SMD:R_0805_2012Metric_Pad1.20x1.40mm_HandSolder, F.Cu at (219.1, 69.8)
- added START1: MX-NoLED, MX_Only:MXOnly-1U-Hotswap, F.Cu at (147.6, 46.8)
- added SW1: SW_Push, Button_Switch_SMD:SW_SPST_SKQG_WithStem, F.Cu at (190.8, 68.6)
- added U1: PRTR5V0U2X, random-keyboard-parts:SOT143B, F.Cu at (228.2, 70.2)
- added U2: ATmega32U4-A, Package_QFP:TQFP-44_10x10mm_P0.8mm, F.Cu at (200.0, 30.2)
- added USB1: HRO-TYPE-C-31-M-12, Type-C:HRO-TYPE-C-31-M-12-HandSoldering, F.Cu at (265.1, 49.1)
- added VOL-L1: RotaryEncoder, Rotary_Encoder:RotaryEncoder_Alps_EC12E_Vertical_H20mm_CircularMountingHoles, F.Cu at (37.1, 70.5)
- added VOL-R1: RotaryEncoder, Rotary_Encoder:RotaryEncoder_Alps_EC12E_Vertical_H20mm_CircularMountingHoles, F.Cu at (243.5, 72.1)
- added Y1: Crystal_GND24_Small, Crystal:Crystal_SMD_3225-4Pin_3.2x2.5mm_HandSoldering, F.Cu at (198.9, 68.1)
Other:
- board text added: "someNesa"

Commit message: i shouldnt have used kicad
mistakes
Parts:
- C1, C2, C3, C4, C5, C6, C7, Fe1, R1, R2, R3, R4, R5, R6, U1, U2, USB1, Y1: moved to B.Cu
- moved J1 263.5 mm to (26.2, 177.0)
- moved C1 141.0 mm to (97.4, 57.9), turned to 180 degrees
- moved R3 141.0 mm to (97.4, 60.9), turned to 180 degrees
- moved SW1 125.3 mm to (277.0, 159.5)
- moved USB1 123.9 mm to (147.6, 9.52)
- moved U2 70.3 mm to (147.6, 77.0), turned to 45 degrees
- moved R5 69.3 mm to (216.2, 54.8), turned to 180 degrees
- moved R1 36.9 mm to (192.8, 66.7), turned to 180 degrees
- moved U1 33.8 mm to (194.4, 70.2), turned to 180 degrees
- moved R2 27.4 mm to (197.6, 66.7), turned to 180 degrees
- moved R4 25.0 mm to (198.8, 69.8), turned to 180 degrees
- moved Y1 20.3 mm to (210.3, 84.9), turned to 180 degrees
- moved C7 17.9 mm to (202.4, 66.8), turned to 180 degrees
- moved R6 15.5 mm to (203.5, 69.8), turned to 180 degrees
- moved VOL-R1 13.7 mm to (250.7, 60.5), turned to 90 degrees
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Other:
- board outline added: 277.8 x 191.3 mm

Commit message: spaghetti
w
Parts:
- moved R6 118.2 mm to (85.7, 79.2), turned to 90 degrees
- moved Fe1 76.3 mm to (153.3, 25.4)
- moved R5 72.0 mm to (144.5, 60.9), turned to -90 degrees
- moved C1 68.1 mm to (164.3, 70.6)
- moved U1 65.2 mm to (147.8, 24.6)
- moved R3 55.6 mm to (136.5, 21.4), turned to 0 degrees
- moved C2 53.3 mm to (158.8, 63.7), turned to -90 degrees
- moved Y1 52.8 mm to (160.0, 69.0), turned to 90 degrees
- moved R4 52.7 mm to (146.8, 60.9), turned to -90 degrees
- moved C7 47.4 mm to (191.5, 20.7)
- moved R1 47.4 mm to (182.0, 20.6)
- moved R2 47.4 mm to (186.7, 20.6)
- moved C4 42.6 mm to (164.6, 67.5)
- moved C3 39.6 mm to (189.9, 42.1), turned to 0 degrees
- moved C5 28.8 mm to (189.9, 47.6), turned to 0 degrees
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Routing:
- net D+: track 0.00 -> 61.3 mm
- net D-: track 0.00 -> 59.8 mm
- net GND: track 0.00 -> 51.8 mm
- net Net-(C4-Pad1): track 0.00 -> 14.9 mm
- net Net-(C1-Pad1): track 0.00 -> 14.4 mm
- net VCC: track 0.00 -> 9.72 mm
- net +5V: track 0.00 -> 7.57 mm
- net Net-(R5-Pad2): track 0.00 -> 2.56 mm
- net Net-(R4-Pad2): track 0.00 -> 1.92 mm
- net Net-(R2-Pad1): track 0.00 -> 0.60 mm
Other:
- outline, holes or cut-outs redrawn

Commit message: done?
done?
Parts:
- removed C5: 0.1u, Capacitor_SMD:C_0805_2012Metric_Pad1.18x1.45mm_HandSolder
- added C8: 0.1u, Capacitor_SMD:C_0805_2012Metric_Pad1.18x1.45mm_HandSolder, B.Cu at (152.2, 77.8)
- J1: moved to B.Cu
- moved J1 202.4 mm to (177.0, 42.1), turned to 180 degrees
- moved SW1 138.7 mm to (198.4, 45.2), turned to 180 degrees
- moved C3 61.6 mm to (138.1, 75.4), turned to 90 degrees
- moved C7 57.0 mm to (150.6, 60.3)
- moved R6 56.4 mm to (142.1, 77.8), turned to 180 degrees
- moved C6 54.8 mm to (136.3, 64.3)
- moved R2 32.7 mm to (154.0, 21.4), turned to 0 degrees
- moved Fe1 27.1 mm to (126.2, 26.9), turned to -90 degrees
- moved R1 25.0 mm to (169.1, 42.1)
- moved R3 4.97 mm to (141.5, 21.4), turned to 180 degrees
- moved R4 3.76 mm to (146.8, 57.1)
- moved R5 3.76 mm to (144.5, 57.1)
Connections:
- net Net-(R4-Pad2) renamed DATAP
- net Net-(R5-Pad2) renamed DATAN
Routing:
- net KEYROW: track 0.00 -> 539.2 mm, vias 0 -> 4
- net GND: track 51.8 -> 264.4 mm, vias 0 -> 6
- net +5V: track 7.57 -> 207.9 mm, vias 0 -> 7
- net START: track 0.00 -> 170.8 mm, vias 0 -> 2
- net VOLLB: track 0.00 -> 157.4 mm, vias 0 -> 4
- net VOLROUT: track 0.00 -> 136.8 mm, vias 0 -> 2
- net COLR: track 0.00 -> 128.9 mm, vias 0 -> 2
- net RESET: track 0.00 -> 105.8 mm, vias 0 -> 3
- net COLL: track 0.00 -> 100.0 mm, vias 0 -> 2
- net VOLRA: track 0.00 -> 95.0 mm
- net VOLRB: track 0.00 -> 86.7 mm, vias 0 -> 2
- net VOLLA: track 0.00 -> 84.5 mm, vias 0 -> 2
- net VOLLOUT: track 0.00 -> 83.5 mm, vias 0 -> 2
- net COLA: track 0.00 -> 82.2 mm, vias 0 -> 2
- net COLD: track 0.00 -> 61.4 mm, vias 0 -> 2
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- added copper zone on B.Cu, net GND
- added copper zone on F.Cu, net GND
