File: sdvx-pcb.kicad_pcb (KiCad board)
At the start: 2 copper layers, 277.8 x 191.3 mm, 29 parts, among them J1 AVR-ISP-6, SW1 SW_Push, U1 PRTR5V0U2X, U2 ATmega32U4-A, Y1 Crystal_GND24_Small

Commit message: rotary encoders
sike not done
Parts:
- renumbered C8 to C2, C2 to C3, C3 to C4, C4 to C5
Routing:
- net VOLROUT: track 136.8 -> 125.8 mm
- net VOLLA: track 84.5 -> 75.1 mm
Other:
- board text added: "BT-A"
- board text added: "BT-B"
- board text added: "BT-C"
- board text added: "BT-D"
- board text added: "FX-L"
- board text added: "FX-R"
- board text added: "Press to reset MCU"
- board text added: "some sdvx controller v1"
- board text removed: "sad sdvx controller v1"
Changed lines of the file:
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@@
   (net 7 "GND")
   (net 8 "+5V")
-  (net 9 "Net-(C4-Pad1)")
+  (net 9 "Net-(C5-Pad1)")
   (net 10 "Net-(C7-Pad1)")
   (net 11 "VCC")
@@
     (property "Sheetname" "")
     (attr smd)
-    (fp_text reference "C2" (at 0 1.68 90) (layer "B.SilkS")
+    (fp_text reference "C3" (at 0 1.68 90) (layer "B.SilkS")
       (effects (font (size 1 1) (thickness 0.15)) (justify mirror))
     )
@@
       (net 7 "GND") (pinfunction "GND") (pintype "power_in"))
     (pad "16" smd rect (at -0.8 -5.7 180) (size 1.5 0.55) (layers "B.Cu" "B.Paste" "B.Mask")
-      (net 9 "Net-(C4-Pad1)") (pinfunction "XTAL2") (pintype "output"))
+      (net 9 "Net-(C5-Pad1)") (pinfunction "XTAL2") (pintype "output"))
     (pad "17" smd rect (at 0 -5.7 180) (size 1.5 0.55) (layers "B.Cu" "B.Paste" "B.Mask")
       (net 6 "Net-(C1-Pad1)") (pinfunction "XTAL1") (pintype "input"))
@@
     (property "Sheetname" "")
     (attr smd)
-    (fp_text reference "C3" (at -0.1 2.10125 90) (layer "B.SilkS")
+    (fp_text reference "C4" (at -0.1 2.10125 90) (layer "B.SilkS")
       (effects (font (size 1 1) (thickness 0.15)) (justify mirror))
     )
@@
     (property "Sheetname" "")
     (attr smd)
-    (fp_text reference "C8" (at 0 1.68) (layer "B.SilkS")
+    (fp_text reference "C2" (at 0 1.68) (layer "B.SilkS")
       (effects (font (size 1 1) (thickness 0.15)) (justify mirror))
     )
@@
     (property "Sheetname" "")
     (attr smd)
-    (fp_text reference "C4" (at 0 1.68) (layer "B.SilkS")
+    (fp_text reference "C5" (at 0 1.68) (layer "B.SilkS")
       (effects (font (size 1 1) (thickness 0.15)) (justify mirror))
     )
@@
     (fp_line (start 1 -0.625) (end -1 -0.625) (layer "B.Fab") (width 0.1))
     (pad "1" smd roundrect (at -1.0375 0 180) (size 1.175 1.45) (layers "B.Cu" "B.Paste" "B.Mask") (roundrect_rratio 0.2127659574)
-      (net 9 "Net-(C4-Pad1)") (pintype "passive"))
+      (net 9 "Net-(C5-Pad1)") (pintype "passive"))
     (pad "2" smd roundrect (at 1.0375 0 180) (size 1.175 1.45) (layers "B.Cu" "B.Paste" "B.Mask") (roundrect_rratio 0.2127659574)
       (net 7 "GND") (pintype "passive"))
@@
       (net 7 "GND") (pinfunction "2") (pintype "passive"))
     (pad "3" smd rect (at 1.45 1.15 90) (size 2.1 1.8) (layers "B.Cu" "B.Paste" "B.Mask")
-      (net 9 "Net-(C4-Pad1)") (pinfunction "3") (pintype "passive"))
+      (net 9 "Net-(C5-Pad1)") (pinfunction "3") (pintype "passive"))
     (pad "4" smd rect (at -1.45 1.15 90) (size 2.1 1.8) (layers "B.Cu" "B.Paste" "B.Mask")
       (net 7 "GND") (pinfunction "4") (pintype "passive"))
@@
   (gr_arc (start 9.525 11.1125) (mid 9.989968 9.989968) (end 11.1125 9.525) (layer "Edge.Cuts") (width 0.1))
   (gr_line (start 287.3375 11.1125) (end 287.327568 199.213778) (layer "Edge.Cuts") (width 0.1))
-  (gr_text "sad sdvx controller v1" (at 200.025 189.70625) (layer "F.Cu")
+  (gr_text "some sdvx controller v1" (at 270.66875 196.85) (layer "F.Cu")
     (effects (font (size 1.5 1.5) (thickness 0.3)))
   )
   (gr_text "someNesa" (at 18.25625 196.85) (layer "F.Cu")
     (effects (font (size 1.5 1.5) (thickness 0.3)))
+  )
+  (gr_text "BT-D" (at 188.11875 116.68125) (layer "F.SilkS")
+    (effects (font (size 1 1) (thickness 0.15)))
+  )
+  (gr_text "FX-R" (at 163.5125 161.925) (layer "F.SilkS")
+    (effects (font (size 1 1) (thickness 0.15)))
+  )
+  (gr_text "BT-C" (at 153.19375 116.68125) (layer "F.SilkS")
+    (effects (font (size 1 1) (thickness 0.15)))
+  )
+  (gr_text "BT-B" (at 118.26875 116.68125) (layer "F.SilkS")
+    (effects (font (size 1 1) (thickness 0.15)))
+  )
+  (gr_text "Press to reset MCU" (at 198.4375 39.6875) (layer "F.SilkS")
+    (effects (font (size 1 1) (thickness 0.15)))
+  )
+  (gr_text "FX-L" (at 93.6625 161.925) (layer "F.SilkS")
+    (effects (font (size 1 1) (thickness 0.15)))
+  )
+  (gr_text "BT-A" (at 83.34375 116.68125) (layer "F.SilkS")
+    (effects (font (size 1 1) (thickness 0.15)))
   )
   (segment (start 130.175 70.64375) (end 109.5375 91.28125) (width 0.254) (layer "F.Cu") (net 1))
@@
   (via (at 124.735589 77.110589) (size 0.8) (drill 0.4) (layers "F.Cu" "B.Cu") (net 35))
   (segment (start 64.67652 77.24223) (end 124.603948 77.24223) (width 0.254) (layer "B.Cu") (net 35))
-  (segment (start 132.5375 72.25) (end 141.9375 72.25) (width 0.254) (layer "B.Cu") (net 35))
   (segment (start 61.39375 80.525) (end 64.67652 77.24223) (width 0.254) (layer "B.Cu") (net 35))
   (segment (start 124.603948 77.24223) (end 124.735589 77.110589) (width 0.254) (layer "B.Cu") (net 35))
@@
   (via (at 130.96875 68.2625) (size 0.8) (drill 0.4) (layers "F.Cu" "B.Cu") (net 39))
   (via (at 136.525 90.4875) (size 0.8) (drill 0.4) (layers "F.Cu" "B.Cu") (net 39))
-  (segment (start 130.98125 68.25) (end 141.9375 68.25) (width 0.254) (layer "B.Cu") (net 39))
   (segment (start 223.24375 90.4875) (end 136.525 90.4875) (width 0.254) (layer "B.Cu") (net 39))
   (segment (start 130.96875 68.2625) (end 130.98125 68.25) (width 0.254) (layer "B.Cu") (net 39))

Commit message: gerber again
gerbers
Parts:
- added C1: 0.1u, Capacitor_SMD:C_0805_2012Metric_Pad1.18x1.45mm_HandSolder, B.Cu at (87.3, 66.7)
- added C2: 0.1u, Capacitor_SMD:C_0805_2012Metric_Pad1.18x1.45mm_HandSolder, B.Cu at (208.0, 69.1)
- added R1: 10k, Resistor_SMD:R_0805_2012Metric_Pad1.20x1.40mm_HandSolder, B.Cu at (77.6, 74.4)
- added R2: 10k, Resistor_SMD:R_0805_2012Metric_Pad1.20x1.40mm_HandSolder, B.Cu at (77.6, 69.8)
- added R4: 10k, Resistor_SMD:R_0805_2012Metric_Pad1.20x1.40mm_HandSolder, B.Cu at (217.3, 73.6)
- added R5: 10k, Resistor_SMD:R_0805_2012Metric_Pad1.20x1.40mm_HandSolder, B.Cu at (217.3, 70.6)
- renumbered C1 to C3, C2 to C4, C3 to C5, C4 to C6, C5 to C7, C6 to C8, C7 to C9, R6 to R10, R1 to R3, R2 to R6, R3 to R7, R4 to R8, R5 to R9, VOL-L1 to VOL-L, VOL-R1 to VOL-R
Connections:
- U2 pad 38: VOLLOUT -> unconnected-(U2-Pad38)
- U2 pad 41: VOLROUT -> unconnected-(U2-Pad41)
- VOL-L pad C: VOLLOUT -> GND
- VOL-R pad C: VOLROUT -> GND
Routing:
- net GND: track 264.4 -> 526.7 mm
- net +5V: track 207.9 -> 343.9 mm, vias 7 -> 10
- net VOLROUT: track 125.8 -> 0.00 mm, vias 2 -> 0
- net VOLLOUT: track 83.5 -> 0.00 mm, vias 2 -> 0
- net VOLLB: track 157.4 -> 219.8 mm, vias 4 -> 6
- net VOLRB: track 86.7 -> 107.0 mm
- net VOLLA: track 75.1 -> 87.9 mm
- net VOLRA: track 95.0 -> 92.0 mm, vias 0 -> 2
Other:
- board text added: "START"
- board text removed: "some sdvx controller v1"

Commit message: where the grounds
WHERE
Parts:
- VOL-L1: renamed from VOL-L; footprint Rotary_Encoder:RotaryEncoder_Alps_EC12E_Vertical_H20mm_CircularMountingHoles -> Rotary_Encoder:RotaryEncoder_Alps_EC11E_Vertical_H20mm_CircularMountingHoles
- VOL-R1: renamed from VOL-R; footprint Rotary_Encoder:RotaryEncoder_Alps_EC12E_Vertical_H20mm_CircularMountingHoles -> Rotary_Encoder:RotaryEncoder_Alps_EC11E_Vertical_H20mm_CircularMountingHoles
Routing:
- net VOLLB: track 219.8 -> 197.1 mm, vias 6 -> 8
- net KEYROW: track 539.2 -> 518.9 mm, vias 4 -> 8
- net D-: track 57.9 -> 71.2 mm
- net D+: track 59.4 -> 72.7 mm
- net VOLRB: track 107.0 -> 100.1 mm
Other:
- board size 277.8 x 191.3 mm -> 195.3 x 154.8 mm
- board text removed: "someNesa"

Commit message: finish
finish?
Connections:
- net START renamed COLSTART
Other:
- outline, holes or cut-outs redrawn
- board text added: "VOL-L"
- board text added: "VOL-R"
- board text added: "someNesa"
Changed lines of the file:
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@@
   (net 21 "DATAN")
   (net 22 "Net-(R6-Pad1)")
-  (net 23 "START")
+  (net 23 "COLSTART")
   (net 24 "VOLLB")
   (net 25 "unconnected-(U2-Pad12)")
@@
     (pad "" np_thru_hole circle locked (at 0 0) (size 3.9878 3.9878) (drill 3.9878) (layers *.Cu *.Mask))
     (pad "1" smd rect locked (at -7.085 -2.54) (size 2.55 2.5) (layers "B.Cu" "B.Paste" "B.Mask")
-      (net 23 "START") (pinfunction "COL") (pintype "passive"))
+      (net 23 "COLSTART") (pinfunction "COL") (pintype "passive"))
     (pad "2" smd rect locked (at 5.842 -5.08) (size 2.55 2.5) (layers "B.Cu" "B.Paste" "B.Mask")
       (net 1 "KEYROW") (pinfunction "ROW") (pintype "passive"))
@@
       (net 28 "VOLRB") (pinfunction "PD2") (pintype "bidirectional"))
     (pad "21" smd rect (at 3.2 -5.7 180) (size 1.5 0.55) (layers "B.Cu" "B.Paste" "B.Mask")
-      (net 23 "START") (pinfunction "PD3") (pintype "bidirectional"))
+      (net 23 "COLSTART") (pinfunction "PD3") (pintype "bidirectional"))
     (pad "22" smd rect (at 4 -5.7 180) (size 1.5 0.55) (layers "B.Cu" "B.Paste" "B.Mask")
       (net 29 "unconnected-(U2-Pad22)") (pinfunction "PD5") (pintype "bidirectional+no_connect"))
@@
     )
   )
-  (gr_line (start 54.76875 164.30625) (end 242.09375 164.30625) (layer "Edge.Cuts") (width 0.1))
-  (gr_arc (start 242.09375 9.525) (mid 244.90008 10.68742) (end 246.0625 13.49375) (layer "Edge.Cuts") (width 0.1))
-  (gr_line (start 50.8 13.49375) (end 50.8 160.3375) (layer "Edge.Cuts") (width 0.1))
-  (gr_arc (start 50.8 13.49375) (mid 51.96242 10.68742) (end 54.76875 9.525) (layer "Edge.Cuts") (width 0.1))
-  (gr_line (start 246.0625 160.3375) (end 246.0625 13.49375) (layer "Edge.Cuts") (width 0.1))
-  (gr_arc (start 54.76875 164.30625) (mid 51.96242 163.14383) (end 50.8 160.3375) (layer "Edge.Cuts") (width 0.1))
-  (gr_arc (start 246.0625 160.3375) (mid 244.90008 163.14383) (end 242.09375 164.30625) (layer "Edge.Cuts") (width 0.1))
-  (gr_line (start 242.09375 9.525) (end 54.76875 9.525) (layer "Edge.Cuts") (width 0.1))
-  (gr_text "BT-D" (at 188.11875 116.68125) (layer "F.SilkS")
-    (effects (font (size 1.5 1.5) (thickness 0.15)))
-  )
-  (gr_text "FX-R" (at 163.5125 161.925) (layer "F.SilkS")
-    (effects (font (size 1.5 1.5) (thickness 0.15)))
-  )
-  (gr_text "BT-C" (at 153.19375 116.68125) (layer "F.SilkS")
-    (effects (font (size 1.5 1.5) (thickness 0.15)))
-  )
-  (gr_text "BT-B" (at 118.26875 116.68125) (layer "F.SilkS")
-    (effects (font (size 1.5 1.5) (thickness 0.15)))
+  (gr_arc (start 52.3875 164.30625) (mid 51.264968 163.841282) (end 50.8 162.71875) (layer "Edge.Cuts") (width 0.1))
+  (gr_line (start 52.3875 164.30625) (end 244.475 164.30625) (layer "Edge.Cuts") (width 0.1))
+  (gr_line (start 50.8 11.1125) (end 50.8 162.71875) (layer "Edge.Cuts") (width 0.1))
+  (gr_arc (start 246.0625 162.71875) (mid 245.597532 163.841282) (end 244.475 164.30625) (layer "Edge.Cuts") (width 0.1))
+  (gr_arc (start 50.8 11.1125) (mid 51.264968 9.989968) (end 52.3875 9.525) (layer "Edge.Cuts") (width 0.1))
+  (gr_line (start 246.0625 162.71875) (end 246.0625 11.1125) (layer "Edge.Cuts") (width 0.1))
+  (gr_arc (start 244.475 9.525) (mid 245.597532 9.989968) (end 246.0625 11.1125) (layer "Edge.Cuts") (width 0.1))
+  (gr_line (start 244.475 9.525) (end 52.3875 9.525) (layer "Edge.Cuts") (width 0.1))
+  (gr_text "BT-D" (at 200.025 120.65) (layer "F.SilkS")
+    (effects (font (size 2 2) (thickness 0.15)))
+  )
+  (gr_text "FX-R" (at 182.5625 135.73125) (layer "F.SilkS")
+    (effects (font (size 2 2) (thickness 0.15)))
+  )
+  (gr_text "BT-C" (at 165.1 120.65) (layer "F.SilkS")
+    (effects (font (size 2 2) (thickness 0.15)))
+  )
+  (gr_text "BT-B" (at 130.175 120.65) (layer "F.SilkS")
+    (effects (font (size 2 2) (thickness 0.15)))
   )
   (gr_text "Press to reset MCU" (at 198.4375 39.6875) (layer "F.SilkS")
     (effects (font (size 1 1) (thickness 0.15)))
   )
-  (gr_text "FX-L" (at 93.6625 161.925) (layer "F.SilkS")
+  (gr_text "someNesa" (at 57.94375 11.90625) (layer "F.SilkS")
     (effects (font (size 1.5 1.5) (thickness 0.15)))
   )
-  (gr_text "BT-A" (at 83.34375 116.68125) (layer "F.SilkS")
-    (effects (font (size 1.5 1.5) (thickness 0.15)))
-  )
-  (gr_text "START" (at 147.6375 50.8) (layer "F.SilkS")
-    (effects (font (size 1.5 1.5) (thickness 0.3)))
+  (gr_text "VOL-R" (at 233.20625 87.3125) (layer "F.SilkS")
+    (effects (font (size 2 2) (thickness 0.15)))
+  )
+  (gr_text "VOL-L" (at 63.94375 87.3125) (layer "F.SilkS")
+    (effects (font (size 2 2) (thickness 0.15)))
+  )
+  (gr_text "FX-L" (at 112.7125 135.73125) (layer "F.SilkS")
+    (effects (font (size 2 2) (thickness 0.15)))
+  )
+  (gr_text "BT-A" (at 95.25 120.65) (layer "F.SilkS")
+    (effects (font (size 2 2) (thickness 0.15)))
+  )
+  (gr_text "START" (at 147.6375 51.59375) (layer "F.SilkS")
+    (effects (font (size 2 2) (thickness 0.3)))
   )
   (segment (start 109.5375 91.28125) (end 100.80625 91.28125) (width 0.254) (layer "F.Cu") (net 1))
