File: sdvx-pcb.kicad_sch (KiCad schematic)
At the start: 14 parts, among them U1 ATmega32U4-A

Commit message: more edits
more edits
Parts:
- added BT-A, BT-B, BT-C, BT-D, FX-L, FX-R: MX-LED, symbol MX_Alps_Hybrid:MX-LED
- added Fe: 500m, symbol Device:Polyfuse_Small
- added J?: AVR-ISP-6, symbol Connector:AVR-ISP-6
- added R? (x2): 5.1k, symbol Device:R_Small
- added U?: PRTR5V0U2X, symbol random-keyboard-parts:PRTR5V0U2X
- added USB?: HRO-TYPE-C-31-M-12, symbol Type-C:HRO-TYPE-C-31-M-12
Connections:
- net +5V: now also Fe.2, J?.2 (VCC)
- net D+: now also U?.2 (IO1), USB?.6 (DP1), USB?.8 (DP2)
- net D-: now also U?.3 (IO2), USB?.5 (DN2), USB?.7 (DN1)
- net GND: now also J?.6 (GND), R?.2, R?.2, U?.1 (GND), USB?.1 (GND), USB?.12 (GND), USB?.13 (SHIELD)
- net RESET: now reaches R?.2, SW?.2, U1.13 (~{RESET})
- net RESET: now also J?.5 (~{RST})
- net BTROW: now reaches U1.1 (PE6)
- net BTROW: now also BT-A.2 (ROW), BT-B.2 (ROW), BT-C.2 (ROW), BT-D.2 (ROW)
- net MOSI: now reaches U1.10 (PB2)
- net MOSI: now also J?.4 (MOSI)
- net MISO: now reaches U1.11 (PB3)
- net MISO: now also J?.1 (MISO)
- net FXROW: now reaches U1.38 (PF5)
- net FXROW: now also FX-L.2 (ROW), FX-R.2 (ROW)
- net SCK: now reaches U1.9 (PB1)
- net SCK: now also J?.3 (SCK)
- new net: R?.1, USB?.10 (CC2)
- new net: R?.1, USB?.4 (CC1)
- new net VCC: Fe.1, USB?.11 (VBUS), USB?.2 (VBUS)
- no-connect marks 2 -> 1
Other:
- moved on the sheet: R?, SW?

Commit message: hmm
hmmm
Parts:
- removed BT-A, BT-B, BT-C, BT-D, FX-L, FX-R: MX-LED, symbol MX_Alps_Hybrid:MX-LED
- added BT-A1, BT-B1, BT-C1, BT-D1: MX-NoLED, MX_Only:MXOnly-1.5U-Hotswap-LED, symbol MX_Alps_Hybrid:MX-NoLED
- added FX-L1, FX-R1: MX-NoLED, MX_Only:MXOnly-2.25U-Hotswap-LED, symbol MX_Alps_Hybrid:MX-NoLED
- C1: renamed from C2; footprint (none) -> Capacitor_SMD:C_0805_2012Metric_Pad1.18x1.45mm_HandSolder
- C2, C3, C5, C6: renamed from C?; footprint (none) -> Capacitor_SMD:C_0805_2012Metric_Pad1.18x1.45mm_HandSolder
- C4: renamed from C3; footprint (none) -> Capacitor_SMD:C_0805_2012Metric_Pad1.18x1.45mm_HandSolder
- C7: renamed from C1; footprint (none) -> Capacitor_SMD:C_0805_2012Metric_Pad1.18x1.45mm_HandSolder
- Fe1: renamed from Fe; footprint (none) -> Fuse:Fuse_1206_3216Metric_Pad1.42x1.75mm_HandSolder
- J1: renamed from J?; footprint (none) -> random-keyboard-parts:Reset_Pretty-Mask
- gave numbers to parts that had none: 9
- renumbered R1 to R6, U1 to U2
Connections:
- net VCC: now also U1.4 (VCC)
- net COLA: now reaches U2.28 (PB4)
- net COLA: now also BT-A1.1 (COL)
- net COLB: now reaches U2.29 (PB5)
- net COLB: now also BT-B1.1 (COL)
- net COLC: now reaches U2.30 (PB6)
- net COLC: now also BT-C1.1 (COL)
- net COLD: now reaches U2.31 (PC6)
- net COLD: now also BT-D1.1 (COL)
- net COLL: now reaches U2.32 (PC7)
- net COLL: now also FX-L1.1 (COL)
- net COLR: now reaches U2.37 (PF6)
- net COLR: now also FX-R1.1 (COL)
- net BTROW renamed KEYROW
- net KEYROW: now also BT-A1.2 (ROW), BT-B1.2 (ROW), BT-C1.2 (ROW), BT-D1.2 (ROW), FX-L1.2 (ROW), FX-R1.2 (ROW)
- net FXROW: no longer names the net of U2.38 (PF5)
- no-connect marks 1 -> 18

Commit message: schematic finish
finished schematic maybe
Parts:
- added VOL-L1, VOL-R1: RotaryEncoder, Rotary_Encoder:RotaryEncoder_Alps_EC12E_Vertical_H20mm_CircularMountingHoles, symbol Device:RotaryEncoder
- BT-A1, BT-B1, BT-C1, BT-D1: footprint MX_Only:MXOnly-1.5U-Hotswap-LED -> MX_Only:MXOnly-1.5U-Hotswap
- FX-L1, FX-R1: footprint MX_Only:MXOnly-2.25U-Hotswap-LED -> MX_Only:MXOnly-2.25U-Hotswap
- R1, R2, R3, R4, R5, R6: footprint (none) -> Resistor_SMD:R_0805_2012Metric_Pad1.20x1.40mm_HandSolder
- SW1: footprint (none) -> Button_Switch_SMD:SW_SPST_SKQG_WithStem
- U1: footprint (none) -> random-keyboard-parts:SOT143B
- USB1: footprint (none) -> Type-C:HRO-TYPE-C-31-M-12-HandSoldering
- Y1: footprint (none) -> Crystal:Crystal_SMD_3225-4Pin_3.2x2.5mm_HandSoldering
Connections:
- net VOLRA: now reaches U2.19 (PD1)
- net VOLRA: now also VOL-R1.A
- net VOLRB: now reaches U2.20 (PD2)
- net VOLRB: now also VOL-R1.B
- net VOLLA: now reaches U2.36 (PF7)
- net VOLLA: now also VOL-L1.A
- net VOLLOUT: now reaches U2.38 (PF5)
- net VOLLOUT: now also VOL-L1.C
- net VOLROUT: now reaches U2.41 (PF0)
- net VOLROUT: now also VOL-R1.C
- net VOLLB: now reaches U2.8 (PB0)
- net VOLLB: now also VOL-L1.B
- no-connect marks 18 -> 12

Commit message: pcb start
start pcb
Parts:
- added START1: MX-NoLED, MX_Only:MXOnly-1U-Hotswap, symbol MX_Alps_Hybrid:MX-NoLED
- renumbered R3 to R1, R1 to R2, R2 to R3
Connections:
- net KEYROW: now also START1.2 (ROW)
- net START: now reaches U2.21 (PD3)
- net START: now also START1.1 (COL)
- no-connect marks 12 -> 11
Other:
- moved on the sheet: R1, SW1

Commit message: spaghetti
w
Changed lines of the file:
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@@
     (stroke (width 0) (type default) (color 0 0 0 0))
+  )
+  (global_label "DP" (shape input) (at 135.89 88.9 270) (fields_autoplaced)
+    (effects (font (size 1.27 1.27)) (justify right))
+    (property "Intersheet References" "${INTERSHEET_REFS}" (id 0) (at 135.8106 93.8531 90)
+      (effects (font (size 1.27 1.27)) (justify right) hide)
+    )
   )
   (global_label "RESET" (shape input) (at 54.61 121.92 0) (fields_autoplaced)
@@
       (effects (font (size 1.27 1.27)) (justify left) hide)
     )
+  )
+  (global_label "DN" (shape input) (at 135.89 86.36 90) (fields_autoplaced)
+    (effects (font (size 1.27 1.27)) (justify left))
+    (property "Intersheet References" "${INTERSHEET_REFS}" (id 0) (at 135.8106 81.3464 90)
+      (effects (font (size 1.27 1.27)) (justify left) hide)
+    )

Commit message: done?
done?
Parts:
- added C8: 0.1u, Capacitor_SMD:C_0805_2012Metric_Pad1.18x1.45mm_HandSolder, symbol Device:C_Small
Connections:
- net +5V: now also C8.1
- net GND: now also C8.2
- net DATAN: now reaches R5.2, U2.3 (D-)
- net DATAP: now reaches R4.2, U2.4 (D+)
Changed lines of the file:
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@@
 (kicad_sch (version 20211123) (generator eeschema)
   (paper "A4")
+  (junction (at 180.34 38.1) (diameter 0) (color 0 0 0 0)
+  )
   (junction (at 99.06 44.45) (diameter 0) (color 0 0 0 0)
   )
@@
   )
   (junction (at 234.95 44.45) (diameter 0) (color 0 0 0 0)
+  )
+  (junction (at 180.34 43.18) (diameter 0) (color 0 0 0 0)
   )
   (junction (at 191.77 43.18) (diameter 0) (color 0 0 0 0)
@@
     (stroke (width 0) (type default) (color 0 0 0 0))
   )
+  (wire (pts (xy 173.99 43.18) (xy 180.34 43.18))
+    (stroke (width 0) (type default) (color 0 0 0 0))
+  )
   (wire (pts (xy 213.36 77.47) (xy 222.25 77.47))
     (stroke (width 0) (type default) (color 0 0 0 0))
@@
   )
   (wire (pts (xy 189.23 43.18) (xy 189.23 46.99))
+    (stroke (width 0) (type default) (color 0 0 0 0))
+  )
+  (wire (pts (xy 173.99 38.1) (xy 180.34 38.1))
     (stroke (width 0) (type default) (color 0 0 0 0))
   )
@@
     )
   )
+  (global_label "DATAN" (shape input) (at 220.98 80.01 270) (fields_autoplaced)
+    (effects (font (size 1.27 1.27)) (justify right))
+    (property "Intersheet References" "${INTERSHEET_REFS}" (id 0) (at 220.9006 88.1683 90)
+      (effects (font (size 1.27 1.27)) (justify right) hide)
+    )
+  )
   (global_label "VOLLA" (shape input) (at 252.73 125.73 0) (fields_autoplaced)
     (effects (font (size 1.27 1.27)) (justify left))
@@
     )
   )
+  (global_label "DATAP" (shape input) (at 220.98 77.47 90) (fields_autoplaced)
+    (effects (font (size 1.27 1.27)) (justify left))
+    (property "Intersheet References" "${INTERSHEET_REFS}" (id 0) (at 220.9006 69.3721 90)
+      (effects (font (size 1.27 1.27)) (justify left) hide)
+    )
+  )
   (global_label "VOLRA" (shape input) (at 67.31 72.39 270) (fields_autoplaced)
     (effects (font (size 1.27 1.27)) (justify right))
@@
     )
     (pin "1")
+  )
+  (symbol (lib_id "Device:C_Small") (at 173.99 40.64 0) (unit 1)
+    (in_bom yes) (on_board yes) (fields_autoplaced)
+    (property "Reference" "C8" (id 0) (at 176.53 39.3762 0)
+      (effects (font (size 1.27 1.27)) (justify left))
+    )
+    (property "Value" "0.1u" (id 1) (at 176.53 41.9162 0)
+      (effects (font (size 1.27 1.27)) (justify left))
+    )
+    (property "Footprint" "Capacitor_SMD:C_0805_2012Metric_Pad1.18x1.45mm_HandSolder" (id 2) (at 173.99 40.64 0)
+      (effects (font (size 1.27 1.27)) hide)
+    )
+    (property "Datasheet" "~" (id 3) (at 173.99 40.64 0)
+      (effects (font (size 1.27 1.27)) hide)
+    )
+    (pin "1")
+    (pin "2")
   )
   (symbol (lib_id "Device:R_Small") (at 123.19 96.52 0) (unit 1)
@@
       (reference "C7") (unit 1) (value "1u") (footprint "Capacitor_SMD:C_0805_2012Metric_Pad1.18x1.45mm_HandSolder")
     )
+    (path "/188dcfc4-9bfc-4f15-9809-ebced3b82686"
+      (reference "C8") (unit 1) (value "0.1u") (footprint "Capacitor_SMD:C_0805_2012Metric_Pad1.18x1.45mm_HandSolder")
+    )
     (path "/ca805011-784e-4a9b-b60c-3f0d892e2f59"

Commit message: rotary encoders
sike not done
Parts:
- removed C5: 0.1u, Capacitor_SMD:C_0805_2012Metric_Pad1.18x1.45mm_HandSolder, symbol Device:C_Small
- added C1, C2: 0.1u, Capacitor_SMD:C_0805_2012Metric_Pad1.18x1.45mm_HandSolder, symbol Device:C_Small
- added R1, R2, R4, R5: 10k, symbol Device:R_Small
- renumbered C1 to C3, C8 to C4, C2 to C5, C3 to C6, C4 to C7, C6 to C8, C7 to C9, R6 to R10, R1 to R3, R2 to R6, R3 to R7, R4 to R8, R5 to R9
Connections:
- net +5V: now also C1.1, C2.1, R1.2, R2.2, R4.2, R5.2
- net GND: now also VOL-L1.C, VOL-R1.C, C1.2, C2.2
- net VOLLA: now also R1.1
- net VOLLB: now also R2.1
- net VOLRA: now also R4.1
- net VOLRB: now also R5.1
- net VOLLOUT: no longer names the net of U2.38 (PF5)
- net VOLLOUT: no longer VOL-L1.C
- net VOLROUT: no longer names the net of U2.41 (PF0)
- net VOLROUT: no longer VOL-R1.C
- no-connect marks 11 -> 13

Commit message: gerber again
gerbers
Parts:
- R1, R2, R4, R5: footprint (none) -> Resistor_SMD:R_0805_2012Metric_Pad1.20x1.40mm_HandSolder
Changed lines of the file:
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@@
       (effects (font (size 1.27 1.27)) (justify left))
     )
-    (property "Footprint" "" (id 2) (at 48.26 77.47 0)
+    (property "Footprint" "Resistor_SMD:R_0805_2012Metric_Pad1.20x1.40mm_HandSolder" (id 2) (at 48.26 77.47 0)
       (effects (font (size 1.27 1.27)) hide)
     )
@@
       (effects (font (size 1.27 1.27)) (justify left))
     )
-    (property "Footprint" "" (id 2) (at 27.94 77.47 0)
+    (property "Footprint" "Resistor_SMD:R_0805_2012Metric_Pad1.20x1.40mm_HandSolder" (id 2) (at 27.94 77.47 0)
       (effects (font (size 1.27 1.27)) hide)
     )
@@
       (effects (font (size 1.27 1.27)) (justify left))
     )
-    (property "Footprint" "" (id 2) (at 80.01 77.47 0)
+    (property "Footprint" "Resistor_SMD:R_0805_2012Metric_Pad1.20x1.40mm_HandSolder" (id 2) (at 80.01 77.47 0)
       (effects (font (size 1.27 1.27)) hide)
     )
@@
       (effects (font (size 1.27 1.27)) (justify left))
     )
-    (property "Footprint" "" (id 2) (at 57.15 77.47 0)
+    (property "Footprint" "Resistor_SMD:R_0805_2012Metric_Pad1.20x1.40mm_HandSolder" (id 2) (at 57.15 77.47 0)
       (effects (font (size 1.27 1.27)) hide)
     )
@@
     )
     (path "/1fdb6b72-cd2d-48c8-85ff-413c71a3a044"
-      (reference "R1") (unit 1) (value "10k") (footprint "")
+      (reference "R1") (unit 1) (value "10k") (footprint "Resistor_SMD:R_0805_2012Metric_Pad1.20x1.40mm_HandSolder")
     )
     (path "/0f801bbb-36b3-49a1-8891-f369fa4479fc"
-      (reference "R2") (unit 1) (value "10k") (footprint "")
+      (reference "R2") (unit 1) (value "10k") (footprint "Resistor_SMD:R_0805_2012Metric_Pad1.20x1.40mm_HandSolder")
     )
     (path "/8b36f513-bb7a-4bb0-b40b-5f0170ecd097"
@@
     )
     (path "/990bfa0d-04b1-4da1-807b-32e7b6684570"
-      (reference "R4") (unit 1) (value "10k") (footprint "")
+      (reference "R4") (unit 1) (value "10k") (footprint "Resistor_SMD:R_0805_2012Metric_Pad1.20x1.40mm_HandSolder")
     )
     (path "/5a69b64f-7868-4fb7-8125-468ed863f9c0"
-      (reference "R5") (unit 1) (value "10k") (footprint "")
+      (reference "R5") (unit 1) (value "10k") (footprint "Resistor_SMD:R_0805_2012Metric_Pad1.20x1.40mm_HandSolder")
     )
     (path "/217a53c7-6ae2-4270-93e6-65726b22b700"
