File: sdvx-pcb.kicad_sch (KiCad schematic)
At the start: 35 parts, among them J1 AVR-ISP-6, SW1 SW_Push, U1 PRTR5V0U2X, U2 ATmega32U4-A, Y1 Crystal_GND24_Small

Commit message: where the grounds
WHERE
Parts:
- VOL-L1, VOL-R1: footprint Rotary_Encoder:RotaryEncoder_Alps_EC12E_Vertical_H20mm_CircularMountingHoles -> Rotary_Encoder:RotaryEncoder_Alps_EC11E_Vertical_H20mm_CircularMountingHoles
Changed lines of the file:
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@@
       (effects (font (size 1.27 1.27)) (justify right))
     )
-    (property "Footprint" "Rotary_Encoder:RotaryEncoder_Alps_EC12E_Vertical_H20mm_CircularMountingHoles" (id 2) (at 34.036 68.58 0)
+    (property "Footprint" "Rotary_Encoder:RotaryEncoder_Alps_EC11E_Vertical_H20mm_CircularMountingHoles" (id 2) (at 34.036 68.58 0)
       (effects (font (size 1.27 1.27)) hide)
     )
@@
       (effects (font (size 1.27 1.27)) (justify right))
     )
-    (property "Footprint" "Rotary_Encoder:RotaryEncoder_Alps_EC12E_Vertical_H20mm_CircularMountingHoles" (id 2) (at 65.786 68.58 0)
+    (property "Footprint" "Rotary_Encoder:RotaryEncoder_Alps_EC11E_Vertical_H20mm_CircularMountingHoles" (id 2) (at 65.786 68.58 0)
       (effects (font (size 1.27 1.27)) hide)
     )
@@
     )
     (path "/2b64f23e-8aa3-423f-98b6-a5736a34d8d1"
-      (reference "VOL-L1") (unit 1) (value "RotaryEncoder") (footprint "Rotary_Encoder:RotaryEncoder_Alps_EC12E_Vertical_H20mm_CircularMountingHoles")
+      (reference "VOL-L1") (unit 1) (value "RotaryEncoder") (footprint "Rotary_Encoder:RotaryEncoder_Alps_EC11E_Vertical_H20mm_CircularMountingHoles")
     )
     (path "/6811e5b7-2e9e-488d-ad26-8cee9006ba67"
-      (reference "VOL-R1") (unit 1) (value "RotaryEncoder") (footprint "Rotary_Encoder:RotaryEncoder_Alps_EC12E_Vertical_H20mm_CircularMountingHoles")
+      (reference "VOL-R1") (unit 1) (value "RotaryEncoder") (footprint "Rotary_Encoder:RotaryEncoder_Alps_EC11E_Vertical_H20mm_CircularMountingHoles")
     )
     (path "/5afcc4d1-6bd3-4c6e-b024-ebc55adcfe5a"

Commit message: finish
finish?
Connections:
- net START renamed COLSTART
Other:
- moved on the sheet: C1, C2
